File: MicUsb_hw/MicUsb.sch (KiCad schematic (older format))
At the start: 7 parts

Commit message: + ioc, sch 20%
Parts:
- removed C? (x6): C, CAP_0603, symbol C
- removed DD?: STM32L151CxTx, symbol STM32L151CxTx
- added C? (x5): 0.1u, CAP_0603, symbol C
- added C? (x5): 1u, CAP_0603, symbol C
- added C?: 10u, CAP_0805, symbol C
- added C? (x2): 20pF, CAP_0603, symbol C
- added DA? (x2): TLV733xx, symbol TLV733xx
- added DD?: STM32L151CCUx, symbol STM32L151CCUx
- added R?: 200R, RES_0603, symbol R
- added XL?: ST_SWD, symbol ST_SWD
- added XL?: CONN_3, symbol CONN_3
- added XTAL?: 12MHz, CRYSTAL, symbol CRYSTAL_H
Connections:
- net labels added: +3.3V_A, +5V, AGND, RX, SWCLK, SWDIO, TX
- wire segments 23 -> 70

Commit message: sch update
Parts:
- added C? (x2): 10n, CAP_0603, symbol C
- added C?: 1u, CAP_0603, symbol C
- added C?: 0.1u, CAP_0603, symbol C
- added L? (x2): BLM15AG102SN1, IND_0402, symbol L
- added Q?: DVIUC6-4SC6, symbol DVIUC6-4SC6
- added R?: 1M, RES_0603, symbol R
- added XL?: USB_MINI_B, symbol USB_MINI_B
Connections:
- net +5V: now also C?.1, C?.1, L?.1, Q?.5 (Vbus)
- net GND: now also C?.1, C?.2, C?.2, C?.2, L?.1, Q?.2 (GND), R?.2
- net D-: now reaches DD?.32 (MISO1/USBDM/PA11)
- net D-: now also Q?.1 (IO1), Q?.6 (IO4), XL?.2 (D-)
- net D+: now reaches DD?.33 (MOSI1/USBDP/PA12)
- net D+: now also Q?.3 (IO2), Q?.4 (IO3), XL?.3 (D+)
- new net SHLD: C?.1, R?.1, XL?.SHLD
- new net USB_IN_1: C?.2, L?.2, XL?.1 (UVcc)
- new net USB_IN_2: L?.2, XL?.4 (UGND), XL?.5 (UID)
Other:
- note added: "Power"
- note added: "USB"
- moved on the sheet: C?, DA?

Commit message: sch update, i need answers!
Parts:
- added C?: 2.2u, CAP_0603, symbol C
- added C?: 47nf, CAP_0603, symbol C
- added C?: 0.47u, CAP_0603, symbol C
- added C? (x3): 0.1u, CAP_0603, symbol C
- added C? (x2): C, CAP_0603, symbol C
- added C?: 1u, CAP_0603, symbol C
- added D?: LED, symbol LED
- added D?: MAX9814, symbol MAX9814
- added DA?: ADS8320, symbol ADS8320
- added F? (x5): Fuse0R, symbol Fuse0R
- added R?: 510R, RES_0603, symbol R
- added R?: 2k, RES_0603, symbol R
- added R?: 100k, RES_0603, symbol R
- added R?: 150k, RES_0603, symbol R
- added R?: RVar, symbol RVar
- added R?: 5R1, RES_0603, symbol R
- added XL?: CONN_AUDIO_SIMPLE, symbol CONN_AUDIO_SIMPLE
Connections:
- net +3.3V_A: now also C?.1, C?.2, D?.2 (~SHDN), D?.5 (VDD), F?.1, R?.1
- net AGND: now also C?.1, C?.1, C?.1, C?.2, C?.2, C?.2, C?.2, D?.11 (NC), D?.4 (NC), D?.7 (GND), D?.PAD (GND), DA?.8 (Vcc), F?.1, F?.2, F?.2, R?.2, R?.2, XL?.1 (COM), XL?.H
- net GND: now also D?.C, F?.2
- net CSIN: now reaches DD?.14 (ADC4/DAC1/CK2/PA4)
- net CSIN: now also DA?.7 (SCK)
- net SCK: now reaches DD?.15 (ADC5/T2C1ETR/DAC2/SCK1/PA5)
- net SCK: now also DA?.2 (+)
- net DOUT: now reaches DD?.16 (ADC6/T10C1/T3C1/MISO1/PA6)
- net DOUT: now also DA?.5 (CS)
- net at DD?.19 (PB1/T3C4/ADC9/VREFOUT): now also R?.1
- net GAIN_CTRL: now reaches DD?.27 (PB14/MISO2/T9C2/ADC20)
- net GAIN_CTRL: now also F?.2
- new net: D?.A, R?.2
- new net: C?.1, D?.1 (CT)
- new net: D?.10 (GAIN), F?.1, F?.1, F?.2
- new net: C?.1, D?.12 (BIAS)
- new net: D?.14 (TH), R?.1, R?.2
- new net: C?.1, D?.3 (CG)
- new net: C?.1, D?.6 (OUT)
- new net: D?.9 (A/R), F?.1
- new net: C?.1, R?.1, XL?.3 (L_IN)
- new net: C?.2, R?.1
- new net: C?.2, C?.2, R?.2
- new net ADC_IN: R?.3
- new net MIC_BIAS: D?.13 (MICBIAS), R?.1, R?.2
- new net MIC_IN: C?.2, D?.8 (MICIN)
- no-connect marks 0 -> 1
Other:
- note added: "Connect TH to MICBIAS\nto disable the AGC."
- note added: "Gain select:\nGAIN = Vdd: gain = 40dB\nGAIN = GND: gain = 50dB"
- moved on the sheet: C?, DA?, DD?, L?, Q?, R?, XL?, XTAL?

Commit message: * ADS
Parts:
- removed C?: C, CAP_0603, symbol C
- removed DA?: ADS8320, symbol ADS8320
- added DA?: ADS8320, symbol ADS8320
- XL?: symbol USB_MINI_B -> USB_MINI_B-RESCUE-MicUsb
Connections:
- net +3.3V_A: now also DA?.1 (Vref)
- net ADC_IN: now also DA?.2 (+)
- net AGND: now also DA?.3 (-), DA?.4 (GND)
- net CSIN: now also DA?.5 (CS)
- net DOUT: now also DA?.6 (DOUT)
- net SCK: now also DA?.7 (SCK)
- net at D?.6 (OUT): now also R?.1
- net at C?.2, C?.2, R?.2: now also DA?.8 (Vcc)
Other:
- moved on the sheet: C?, D?, DD?, F?, R?, XL?, XTAL?

Commit message: * annotate, footprints
Parts:
- C1, C10, C12, C13, C15, C16, C17, C18, C19, C2, C20, C21, C22, C23, C24, C25, C3, C4, C5, C6, C7, C8, C9: renamed from C?; footprint CAP_0603 -> Capacitors:CAP_0603
- C11: renamed from C?; value C -> 1u; footprint CAP_0603 -> Capacitors:CAP_0603
- C14: renamed from C?; footprint CAP_0805 -> Capacitors:CAP_0805
- D1: renamed from D?; footprint (none) -> QFN_DFN:DFN14
- D2: renamed from D?; footprint (none) -> LEDs:LED_0603
- DA1, DA2: renamed from DA?; footprint (none) -> SOT:SOT23-5
- F1, F2, F3, F4, F5: renamed from F?; footprint (none) -> Resistors:RES_0603_SOLDERFUSE
- L1, L2: renamed from L?; footprint IND_0402 -> Inductors:IND_0402
- Q1: renamed from Q?; footprint (none) -> SOT:SOT23-6
- R1, R2, R3, R4, R6, R7, R8: renamed from R?; footprint RES_0603 -> Resistors:RES_0603
- R5: renamed from R?; value RVar -> 20k; footprint (none) -> Resistors:VAR_PTV09A-4
- XL1: renamed from XL?; footprint (none) -> Connectors:USBmicro_MOLEX_WM17142
- XL2: renamed from XL?; footprint (none) -> Connectors:AUDIO_CKX3_5_30
- XL3: renamed from XL?; footprint (none) -> Connectors:PLS-4
- XL4: renamed from XL?; footprint (none) -> Connectors:PLS-3
- XTAL1: renamed from XTAL?; footprint CRYSTAL -> Quartz:0503x4-4
- gave numbers to parts that had none: 2
Connections:
- no-connect marks 1 -> 26

Commit message: small scheme updates
Parts:
- removed DD1: STM32L151CCUx, symbol STM32L151CCUx
- added D3, D4, D5: LED, LEDs:LED_0603, symbol LED
- added DD1: STM32L151CCTx, LQFP_TQFP:LQFP48, symbol STM32L151CCTx
- added F6: Fuse0R, Resistors:RES_0603_SOLDERFUSE, symbol Fuse0R
- added R10, R11, R9: 1k, Resistors:RES_0603, symbol R
- added SW1: BUTTON, BtnsSwitches:BTN_6x6, symbol BUTTON
- DA3: footprint (none) -> SO_DIL_TSSOP:MSOP8
- R6: value 510R -> 1k
Connections:
- net +3.3V: now also DD1.1 (VDD), DD1.24 (VDD1), DD1.36 (VDD2), DD1.48 (VDD3), DD1.9 (VDDA)
- net ADC_IN: now also F6.1
- net CSIN: now also DD1.14 (ADC4/DAC1/CK2/PA4)
- net D+: now also DD1.33 (MOSI1/USBDP/PA12)
- net D-: now also DD1.32 (MISO1/USBDM/PA11)
- net DOUT: now also DD1.16 (ADC6/T10C1/T3C1/MISO1/PA6)
- net GAIN_CTRL: now also DD1.27 (PB14/MISO2/T9C2/ADC20)
- net GND: now also D3.C, D4.C, D5.C, DD1.23 (VSS1), DD1.35 (VSS2), DD1.44 (BOOT0), DD1.47 (VSS3), DD1.8 (VSSA), SW1.1
- net RX: now also DD1.31 (RX1/PA10)
- net SCK: now also DD1.15 (ADC5/T2C1ETR/DAC2/SCK1/PA5)
- net SWCLK: now also DD1.37 (SWCLK/PA14)
- net SWDIO: now also DD1.34 (SWDIO/PA13)
- net TX: now also DD1.30 (TX1/PA9)
- net at R6.1: now also DD1.19 (PB1/T3C4/ADC9/VREFOUT)
- net at C25.1, XTAL1.2: now also DD1.5 (OSCIN/PH0)
- net at R8.2: now also DD1.6 (OSCOUT/PH1)
- net at D1.6 (OUT), R5.1: now also F6.2
- new net: DD1.18 (PB0/T3C3/ADC8/VREFOUT), R9.1
- new net: D3.A, R9.2
- new net: DD1.40 (PB4/T3C1/MISO1/MISO3), R10.1
- new net: D4.A, R10.2
- new net: DD1.41 (PB5/T3C2/MOSI1/MOSI3), R11.1
- new net: D5.A, R11.2
- new net: DD1.42 (PB6/SCL1/T4C1/TX1), SW1.2
- no-connect marks 26 -> 22
Other:
- moved on the sheet: D2, R5, R6

Commit message: + LP filter, i need answers!
Parts:
- added C? (x3): 1n, CAP_0603, symbol C
- added C?: 1.8n, CAP_0603, symbol C
- added C?: 12n, CAP_0603, symbol C
- added C?: 47n, CAP_0603, symbol C
- added C?: 10n, CAP_0603, symbol C
- added C?: 4.7u, CAP_0603, symbol C
- added DA? (x4): Generic_14pin, symbol Generic_14pin
- added R?: 75k, RES_0603, symbol R
- added R?: 39k, RES_0603, symbol R
- added R?: 9.1k, RES_0603, symbol R
- added R?: 15k, RES_0603, symbol R
- added R?: 3k, RES_0603, symbol R
- added R?: 4.7k, RES_0603, symbol R
- added R?: 75R, RES_0603, symbol R
- added R?: 120R, RES_0603, symbol R
Connections:
- net +3.3V_A: now also DA?.4 (V+), DA?.4 (V+), DA?.4 (V+), DA?.4 (V+)
- net AGND: now also C?.2, C?.2, C?.2, C?.2, DA?.11 (V-), DA?.11 (V-), DA?.11 (V-), DA?.11 (V-)
- new net: C?.1, DA?.1, DA?.2 (-), R?.2 (x3)
- new net: C?.1, DA?.3 (+), R?.1 (x4)
- new net: C?.2, R?.1, R?.2 (x4)
- new net: C?.1, DA?.1, DA?.2 (-)
Other:
- moved on the sheet: C10, C11, C12, C13, C14, C15, C16, C17, C18, C19, C20, C21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

Commit message: *filter
Parts:
- C?: value 1.8n -> 2.2n
- C?: value 1n -> 2.2n
- C?: value 10n -> 15n
- R?: value 4.7k -> 3k
- R?: value 75R -> 69.8R
- R?: value 120R -> 130R
Connections:
- net at C?.1, R?.2: now also DA?.6 (-), DA?.7; no longer DA?.1, DA?.2 (-)
- net at C?.1, R?.1: now also DA?.5 (+); no longer DA?.3 (+)
- net at C?.1, R?.2: now also DA?.8, DA?.9 (-); no longer DA?.1, DA?.2 (-)
- net at C?.1, R?.1: now also DA?.10 (+); no longer DA?.3 (+)
- net at C?.1, R?.1: now also DA?.12 (+); no longer DA?.3 (+)
- new net: C?.1, DA?.13 (-), DA?.14
Changed lines of the file:
@@
 P 6950 4600
 F 0 "C?" V 6900 4450 50  0000 L CNN
-F 1 "1.8n" V 6900 4650 50  0000 L CNN
+F 1 "2.2n" V 6900 4650 50  0000 L CNN
 F 2 "CAP_0603" V 7050 4450 28  0000 C BNN
 F 3 "" H 6950 4600 60  0000 C CNN
@@
 $Comp
 L Generic_14pin DA?
-U 1 1 5653AAF6
+U 2 1 5653AAF6
 P 10100 5300
 F 0 "DA?" H 10150 5500 60  0000 C CNN
@@
 F 2 "" H 10100 5300 60  0000 C CNN
 F 3 "" H 10100 5300 60  0000 C CNN
-	1    10100 5300
+	2    10100 5300
 	1    0    0    -1
 $EndComp
@@
 $Comp
 L Generic_14pin DA?
-U 1 1 5653E042
+U 3 1 5653E042
 P 12500 5300
 F 0 "DA?" H 12550 5500 60  0000 C CNN
@@
 F 2 "" H 12500 5300 60  0000 C CNN
 F 3 "" H 12500 5300 60  0000 C CNN
-	1    12500 5300
+	3    12500 5300
 	1    0    0    -1
 $EndComp
@@
 P 11550 5200
 F 0 "R?" V 11630 5050 50  0000 C CNN
-F 1 "4.7k" V 11550 5200 50  0000 C CNN
+F 1 "3k" V 11550 5200 50  0000 C CNN
 F 2 "RES_0603" V 11630 5300 28  0000 C CNN
 F 3 "" H 11550 5200 60  0000 C CNN
@@
 P 11900 5500
 F 0 "C?" H 11800 5400 50  0000 L CNN
-F 1 "1n" H 11800 5600 50  0000 L CNN
+F 1 "2.2n" H 11800 5600 50  0000 L CNN
 F 2 "CAP_0603" V 12000 5350 28  0000 C BNN
 F 3 "" H 11900 5500 60  0000 C CNN
@@
 $Comp
 L Generic_14pin DA?
-U 1 1 56540686
+U 4 1 56540686
 P 14900 5300
 F 0 "DA?" H 14950 5500 60  0000 C CNN
@@
 F 2 "" H 14900 5300 60  0000 C CNN
 F 3 "" H 14900 5300 60  0000 C CNN
-	1    14900 5300
+	4    14900 5300
 	1    0    0    -1
 $EndComp
@@
 P 13350 5200
 F 0 "R?" V 13430 5050 50  0000 C CNN
-F 1 "75R" V 13350 5200 50  0000 C CNN
+F 1 "69.8R" V 13350 5200 50  0000 C CNN
 F 2 "RES_0603" V 13430 5300 28  0000 C CNN
 F 3 "" H 13350 5200 60  0000 C CNN
@@
 P 13950 5200
 F 0 "R?" V 14030 5050 50  0000 C CNN
-F 1 "120R" V 13950 5200 50  0000 C CNN
+F 1 "130R" V 13950 5200 50  0000 C CNN
 F 2 "RES_0603" V 14030 5300 28  0000 C CNN
 F 3 "" H 13950 5200 60  0000 C CNN
@@
 P 14300 5500
 F 0 "C?" H 14200 5400 50  0000 L CNN
-F 1 "10n" H 14200 5600 50  0000 L CNN
+F 1 "15n" H 14200 5600 50  0000 L CNN
 F 2 "CAP_0603" V 14400 5350 28  0000 C BNN
 F 3 "" H 14300 5500 60  0000 C CNN
