File: MicUsb_hw/MicUsb.kicad_pcb (KiCad board)
At the start: 2 copper layers, 77 parts, among them Q1 DVIUC6-4SC6, SW1 BUTTON

Commit message: * pcb 50%
Parts:
- added TP1: TESTPOINT, PCB:TESTPOINT_1MM, F.Cu at (135.0, 83.5)
- added TP2: TESTPOINT, PCB:TESTPOINT_1MM, F.Cu at (133.2, 83.5)
- added TP3: TESTPOINT, PCB:TESTPOINT_1MM, F.Cu at (131.6, 83.7)
- D2, D3, D4, D5: footprint LEDs:LED_0603 -> LEDs:LED_Through-Hole-3mm
- moved R5 122.6 mm to (158.4, 115.5), turned to 180 degrees
- moved DA4 101.1 mm to (137.6, 113.5), turned to 90 degrees
- moved F2 99.7 mm to (158.2, 105.2), turned to 90 degrees
- moved F6 97.0 mm to (159.6, 111.4)
- moved XL3 88.8 mm to (115.8, 115.2), turned to 90 degrees
- moved R4 88.4 mm to (157.7, 96.0)
- moved D4 85.7 mm to (149.8, 81.8), turned to 90 degrees
- moved D1 85.3 mm to (155.5, 101.2), turned to 270 degrees
- moved DA3 83.7 mm to (124.1, 114.4)
- moved C1 83.6 mm to (116.2, 95.5), turned to 180 degrees
- moved DA2 74.9 mm to (107.6, 115.3), turned to 270 degrees
- moved SW1 74.8 mm to (158.4, 82.2)
- moved XTAL1 74.7 mm to (142.3, 92.2), turned to 270 degrees
- moved C32 74.6 mm to (130.2, 118.7), turned to 180 degrees
- moved R3 74.6 mm to (157.7, 97.8), turned to 180 degrees
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Other:
- board outline added: 66.2 x 44 mm
- net class Default: trace_width 0.25 -> 0.2; via_dia 0.6 -> 0.8
- net class Wide added: clearance 0.2, trace_width 0.5, via_dia 0.8, via_drill 0.4

Commit message: + plot
Parts:
- moved C10 43.9 mm to (130.4, 80.5), turned to 180 degrees
- moved DA2 43.1 mm to (134.4, 81.7), turned to 180 degrees
- moved C13 38.4 mm to (134.6, 84.9), turned to 180 degrees
- moved F1 34.8 mm to (130.4, 85.0), turned to 180 degrees
- moved C9 31.9 mm to (121.7, 80.5), turned to 180 degrees
- moved DA1 30.9 mm to (125.8, 81.8), turned to 180 degrees
- moved R10 28.3 mm to (150.0, 86.0)
- moved C12 26.3 mm to (125.9, 85.1), turned to 180 degrees
- moved F4 21.1 mm to (148.8, 108.7)
- moved F3 21.1 mm to (148.8, 105.2)
- moved F5 20.8 mm to (145.6, 105.8)
- moved R9 17.6 mm to (146.0, 86.1)
- moved C6 10.3 mm to (162.3, 97.3), turned to 270 degrees
- moved C15 7.01 mm to (125.0, 91.0), turned to 180 degrees
- moved C21 6.83 mm to (137.9, 93.2), turned to 0 degrees
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Routing:
- net GND: track 0.00 -> 267.3 mm, vias 0 -> 39
- net AGND: track 0.00 -> 260.2 mm, vias 0 -> 36
- net +3.3V: track 0.00 -> 84.4 mm, vias 0 -> 3
- net +3.3V_A: track 0.00 -> 82.1 mm, vias 0 -> 3
- net Net-(DD1-Pad42): track 0.00 -> 43.9 mm, vias 0 -> 2
- net +5V: track 0.00 -> 41.5 mm, vias 0 -> 3
- net Net-(DD1-Pad40): track 0.00 -> 34.4 mm, vias 0 -> 2
- net /SHLD: track 0.00 -> 33.0 mm, vias 0 -> 4
- net /GAIN_CTRL: track 0.00 -> 28.4 mm, vias 0 -> 2
- net /SCK: track 0.00 -> 24.9 mm, vias 0 -> 2
- net /SWCLK: track 0.00 -> 24.7 mm, vias 0 -> 1
- net /CSIN: track 0.00 -> 24.6 mm
- net /DOUT: track 0.00 -> 24.2 mm
- net /RX: track 0.00 -> 23.2 mm, vias 0 -> 1
- net /TX: track 0.00 -> 21.0 mm, vias 0 -> 1
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- added copper zone on B.Cu, net GND
- added copper zone on F.Cu, net GND
Other:
- board size 66.2 x 44 mm -> 61 x 44 mm
- net class Default: via_drill 0.4 -> 0.3
- net class Wide: via_drill 0.4 -> 0.3

Commit message: plot again
Routing:
- added copper zone on B.Cu, net AGND
- added copper zone on F.Cu, net AGND
Changed lines of the file:
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@@
   (general
     (links 193)
-    (no_connects 5)
-    (area 99.949999 77.755 169.174011 122.500001)
+    (no_connects 0)
+    (area 99.949999 78.24346 169.174011 122.500001)
     (thickness 1.6)
     (drawings 30)
@@
   (page A4)
   (layers
-    (0 F.Cu signal hide)
-    (31 B.Cu signal hide)
+    (0 F.Cu signal)
+    (31 B.Cu signal)
     (32 B.Adhes user)
     (33 F.Adhes user)
@@
     (visible_elements 7FFFF7FF)
     (pcbplotparams
-      (layerselection 0x00030_80000001)
-      (usegerberextensions false)
+      (layerselection 0x010e0_80000001)
+      (usegerberextensions true)
       (excludeedgelayer true)
       (linewidth 0.100000)
@@
       (outputformat 1)
       (mirror false)
-      (drillshape 1)
+      (drillshape 0)
       (scaleselection 1)
-      (outputdirectory ""))
+      (outputdirectory Gerber/))
   )
   (net 0 "")
@@
     (connect_pads (clearance 0.3))
     (min_thickness 0.254)
-    (fill yes (arc_segments 16) (thermal_gap 0.508) (thermal_bridge_width 0.508))
+    (fill yes (arc_segments 32) (thermal_gap 0.3) (thermal_bridge_width 0.508))
     (polygon
       (pts
-        (xy 166.1 122.5) (xy 105 122.4) (xy 105.05 94.9) (xy 110.65 94.95) (xy 110.65 87.15)
-        (xy 105.05 87.15) (xy 105.05 78.45) (xy 166.15 78.45) (xy 166.1 122.5)
+        (xy 105 78.5) (xy 166 78.5) (xy 166 86) (xy 152 86) (xy 145.5 95)
+        (xy 145.5 105) (xy 118 105) (xy 118 122.5) (xy 105 122.5) (xy 105 95)
       )
     )
@@
     (connect_pads (clearance 0.3))
     (min_thickness 0.254)
-    (fill yes (arc_segments 16) (thermal_gap 0.508) (thermal_bridge_width 0.508))
+    (fill yes (arc_segments 32) (thermal_gap 0.3) (thermal_bridge_width 0.508))
     (polygon
       (pts
-        (xy 105 78.45) (xy 166.1 78.4) (xy 166.1 122.45) (xy 104.95 122.4) (xy 105 94.95)
-        (xy 110.6 94.9) (xy 110.55 87.15) (xy 105 87.15) (xy 105.05 78.45)
+        (xy 105 78.5) (xy 166 78.5) (xy 166 86) (xy 152 86) (xy 145.5 95)
+        (xy 145.5 105) (xy 118 105) (xy 118 122.5) (xy 105 122.5)
+      )
+    )
+  )
+  (zone (net 6) (net_name AGND) (layer F.Cu) (hatch edge 0.508)
+    (connect_pads (clearance 0.3))
+    (min_thickness 0.254)
+    (fill yes (arc_segments 32) (thermal_gap 0.3) (thermal_bridge_width 0.508))
+    (polygon
+      (pts
+        (xy 166 86.5) (xy 166 122.5) (xy 118.5 122.5) (xy 118.5 105.5) (xy 146 105.5)
+        (xy 146 95.5) (xy 152.5 86.5) (xy 154.5 86.5)
+      )
+    )
+  )
+  (zone (net 6) (net_name AGND) (layer B.Cu) (hatch edge 0.508)
+    (connect_pads (clearance 0.3))
+    (min_thickness 0.254)
+    (fill yes (arc_segments 32) (thermal_gap 0.3) (thermal_bridge_width 0.508))
+    (polygon
+      (pts
+        (xy 166 86.5) (xy 166 122.5) (xy 118.5 122.5) (xy 118.5 105.5) (xy 146 105.5)
+        (xy 146 95.5) (xy 152.5 86.5)
       )
     )
